File: SMD-NE555.kicad_sch (KiCad schematic)
At the start: 13 parts, among them IC1 NE555D, J1 Conn_01x02_Pin, J2 Conn_01x01_Pin

Commit message: molex to pinheader2.54 1x02
Parts:
- J1: footprint Connector_Molex:Molex_KK-254_AE-6410-02A_1x02_P2.54mm_Vertical -> Connector_PinHeader_2.54mm:PinHeader_1x02_P2.54mm_Vertical
Changed lines of the file:
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@@
 			)
 		)
-		(property "Footprint" "Connector_Molex:Molex_KK-254_AE-6410-02A_1x02_P2.54mm_Vertical"
+		(property "Footprint" "Connector_PinHeader_2.54mm:PinHeader_1x02_P2.54mm_Vertical"
 			(at 57.15 66.04 0)
 			(effects
